File: tusb320-breakout-board.kicad_sch (KiCad schematic)
At the start: 7 parts, among them J1 USB-C Receptacle (USB 2.0), J2 Left Header Pins, J3 Right Header Pins, U1 TUSB320

Commit message: Add jumper to connect VBUS to VBUS_DET
Parts:
- added R2: 0K, Resistor_SMD:R_0402_1005Metric, symbol Device:R_US
Connections:
- net at C1.2, J1.A4 (VBUS), J1.A9 (VBUS)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: now also R2.1
- net at J2.7 (Pin_7), R1.1: now also R2.2
Changed lines of the file:
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@@
     (company "ide")
   )
+  (junction (at 146.05 52.07) (diameter 0) (color 0 0 0 0)
+  )
   (junction (at 146.05 104.14) (diameter 0) (color 0 0 0 0)
   )
@@
   )
   (junction (at 168.91 111.76) (diameter 0) (color 0 0 0 0)
+  )
+  (junction (at 173.99 64.77) (diameter 0) (color 0 0 0 0)
   )
   (junction (at 186.69 57.15) (diameter 0) (color 0 0 0 0)
@@
     (stroke (width 0) (type default) (color 0 0 0 0))
   )
+  (wire (pts (xy 146.05 52.07) (xy 146.05 64.77))
+    (stroke (width 0) (type default) (color 0 0 0 0))
+  )
   (wire (pts (xy 193.04 80.01) (xy 99.06 80.01))
     (stroke (width 0) (type default) (color 0 0 0 0))
@@
     (stroke (width 0) (type default) (color 0 0 0 0))
   )
+  (wire (pts (xy 153.67 64.77) (xy 173.99 64.77))
+    (stroke (width 0) (type default) (color 0 0 0 0))
+  )
   (wire (pts (xy 120.65 82.55) (xy 120.65 64.77))
     (stroke (width 0) (type default) (color 0 0 0 0))
@@
     (stroke (width 0) (type default) (color 0 0 0 0))
   )
+  (wire (pts (xy 146.05 52.07) (xy 193.04 52.07))
+    (stroke (width 0) (type default) (color 0 0 0 0))
+  )
   (wire (pts (xy 186.69 57.15) (xy 186.69 119.38))
     (stroke (width 0) (type default) (color 0 0 0 0))
@@
     (stroke (width 0) (type default) (color 0 0 0 0))
   )
-  (wire (pts (xy 104.14 52.07) (xy 193.04 52.07))
+  (wire (pts (xy 104.14 52.07) (xy 146.05 52.07))
     (stroke (width 0) (type default) (color 0 0 0 0))
   )
@@
     (pin "9")
   )
+  (symbol (lib_id "Device:R_US") (at 149.86 64.77 90) (unit 1)
+    (in_bom yes) (on_board yes)
+    (property "Reference" "R2" (id 0) (at 151.13 59.69 90)
+      (effects (font (size 1.27 1.27)) (justify left))
+    )
+    (property "Value" "0K" (id 1) (at 151.13 62.23 90)
+      (effects (font (size 1.27 1.27)) (justify left))
+    )
+    (property "Footprint" "Resistor_SMD:R_0402_1005Metric" (id 2) (at 150.114 63.754 90)
+      (effects (font (size 1.27 1.27)) hide)
+    )
+    (property "Datasheet" "~" (id 3) (at 149.86 64.77 0)
+      (effects (font (size 1.27 1.27)) hide)
+    )
+    (pin "1")
+    (pin "2")
+  )
   (symbol (lib_id "Device:C") (at 104.14 88.9 180) (unit 1)
     (in_bom yes) (on_board yes)
@@
       (reference "R1") (unit 1) (value "887K") (footprint "Resistor_SMD:R_0402_1005Metric")
     )
+    (path "/d92bc9c2-6b7d-4dd5-95b2-491cd1482b73"
+      (reference "R2") (unit 1) (value "0K") (footprint "Resistor_SMD:R_0402_1005Metric")
+    )
     (path "/809878de-1697-4471-b05f-132bef652e86"
